File: astabile-kippstufe.sch (KiCad schematic (older format))
At the start: 14 parts, among them X1 +UB, X2 0V

Commit message: v19.0.2 inkl doku und gerber
Parts:
- added Logo1: Silk, astabile-kippstufe:HTL-Steyr-Logo_4x4mm_SilkScreen, symbol Device:R
- added Logo2: Copper, astabile-kippstufe:HTL-Steyr-Logo_4x4mm_Copper, symbol Device:R
- C1, C2: footprint astabile-kippstufe:CP_Radial_D10.0mm_P5.00mm -> astabile-kippstufe:CP_Radial_D10.0mm_P5.00mm_P2.50mm
Other:
- moved on the sheet: C1, C2, D1, D2, D3, D4, R1, R2, R3, R4, V1, V2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

Commit message: Montagelöcher
Parts:
- added H1, H2, H3, H4: MountingHole, MountingHole:MountingHole_3.2mm_M3, symbol Mechanical:MountingHole
Changed lines of the file:
@@
+	1    0    0    -1
+$EndComp
+$Comp
+L Mechanical:MountingHole H1
+U 1 1 5EF07E87
+P 12300 5850
+F 0 "H1" H 12400 5896 50  0000 L CNN
+F 1 "MountingHole" H 12400 5805 50  0000 L CNN
+F 2 "MountingHole:MountingHole_3.2mm_M3" H 12300 5850 50  0001 C CNN
+F 3 "~" H 12300 5850 50  0001 C CNN
+	1    12300 5850
+	1    0    0    -1
+$EndComp
+$Comp
+L Mechanical:MountingHole H2
+U 1 1 5EF0C084
+P 12300 6150
+F 0 "H2" H 12400 6196 50  0000 L CNN
+F 1 "MountingHole" H 12400 6105 50  0000 L CNN
+F 2 "MountingHole:MountingHole_3.2mm_M3" H 12300 6150 50  0001 C CNN
+F 3 "~" H 12300 6150 50  0001 C CNN
+	1    12300 6150
+	1    0    0    -1
+$EndComp
+$Comp
+L Mechanical:MountingHole H3
+U 1 1 5EF0C567
+P 12300 6450
+F 0 "H3" H 12400 6496 50  0000 L CNN
+F 1 "MountingHole" H 12400 6405 50  0000 L CNN
+F 2 "MountingHole:MountingHole_3.2mm_M3" H 12300 6450 50  0001 C CNN
+F 3 "~" H 12300 6450 50  0001 C CNN
+	1    12300 6450
+	1    0    0    -1
+$EndComp
+$Comp
+L Mechanical:MountingHole H4
+U 1 1 5EF0C807
+P 12300 6700
+F 0 "H4" H 12400 6746 50  0000 L CNN
+F 1 "MountingHole" H 12400 6655 50  0000 L CNN
+F 2 "MountingHole:MountingHole_3.2mm_M3" H 12300 6700 50  0001 C CNN
+F 3 "~" H 12300 6700 50  0001 C CNN
+	1    12300 6700
 	1    0    0    -1
 $EndComp
